Commit message: Apply workaround on line issues

File: world_desc/lks_arena.main.xacro (robot description, xacro)
@@ -50,5 +50,5 @@
     </visual>
     <collision>
-      <origin xyz="0 0 0"/>
+      <origin xyz="0 0 -0.1"/>
       <geometry>
         <box size="1.8 0.054 0.0001"/>
@@ -70,5 +70,5 @@
     </visual>
     <collision>
-      <origin xyz="0 0 0"/>
+      <origin xyz="0 0 -0.1"/>
       <geometry>
         <box size="1.8 0.054 0.0001"/>
@@ -90,5 +90,5 @@
     </visual>
     <collision>
-      <origin xyz="0 0 0"/>
+      <origin xyz="0 0 -0.1"/>
       <geometry>
         <box size="1.8 0.054 0.0001"/>
@@ -110,5 +110,5 @@
     </visual>
     <collision>
-      <origin xyz="0 0 0"/>
+      <origin xyz="0 0 -0.1"/>
       <geometry>
         <box size="1.8 0.054 0.0001"/>
