Commit message: Added container boxes and lines

File: world_desc/lks_arena.include.xacro (robot description, xacro)
@@ -39,4 +39,30 @@
     </gazebo>
   </xacro:macro>
+  <!-- CONTAINER BOX GENERATION -->
+  <xacro:macro name="cont_box" params="name">
+    <link name="${name}">
+      <visual>
+        <origin xyz="0 0 0"/>
+        <geometry>
+          <box size="0.3 0.3 0.3"/>
+        </geometry>
+        <material name="white">
+          <color rgba="1 1 1 1"/>
+        </material>
+      </visual>
+      <collision>
+        <origin xyz="0 0 0"/>
+        <geometry>
+          <box size="0.3 0.3 0.3"/>
+        </geometry>
+      </collision>
+      <xacro:inertial_box mass="0.3" x="0.3" y="0.3" z="0.3">
+        <origin xyz="0 0 0"/>
+      </xacro:inertial_box>
+    </link>
+    <gazebo reference="${name}">
+      <material>Gazebo/White</material>
+    </gazebo>
+  </xacro:macro>
   <!-- OBJECT-BASE JOINT GENERATION -->
   <xacro:macro name="wall_joint" params="wall *origin">
@@ -47,3 +73,62 @@
     </joint>
   </xacro:macro>
+  <!-- 4 CONTAINER BOX CLUSTER GENERATION -->
+  <xacro:macro name="cont_box_4" params="name0 name1 name2 name3 x y">
+    <xacro:wall_joint wall="${name0}">
+      <origin xyz="${6 - x - 0.15} ${3 - y - 0.3 - 0.3} ${0.15 + 0.027}"/>
+    </xacro:wall_joint>
+    <xacro:wall_joint wall="${name1}">
+      <origin xyz="${6 - x - 0.15} ${3 - y - 0.15} ${0.15 + 0.027}"/>
+    </xacro:wall_joint>
+    <xacro:wall_joint wall="${name2}">
+      <origin xyz="${6 - x - 0.6} ${3 - y - 0.15} ${0.15 + 0.027}"/>
+    </xacro:wall_joint>
+    <xacro:wall_joint wall="${name3}">
+      <origin xyz="${6 - x - 0.6} ${3 - y - 0.3 - 0.3} ${0.15 + 0.027}"/>
+    </xacro:wall_joint>
+  </xacro:macro>
+  <!-- 2 CONTAINER BOX CLUSTER GENERATION -->
+  <xacro:macro name="cont_box_2" params="name0 name1 x y">
+    <xacro:wall_joint wall="${name0}">
+      <origin xyz="${6 - x - 0.15} ${3 - y - 0.15} ${0.15 + 0.027}"/>
+    </xacro:wall_joint>
+    <xacro:wall_joint wall="${name1}">
+      <origin xyz="${6 - x - 0.6} ${3 - y - 0.15} ${0.15 + 0.027}"/>
+    </xacro:wall_joint>
+  </xacro:macro>
+  <!-- LINE GENERATION -->
+  <xacro:macro name="make_line" params="name">
+    <link name="${name}">
+      <visual>
+        <origin xyz="0 0 0"/>
+        <geometry>
+          <box size="0.45 0.054 0.0001"/>
+        </geometry>
+        <material name="black">
+          <color rgba="0.01 0.01 0.01 1"/>
+        </material>
+      </visual>
+      <collision>
+        <origin xyz="0 0 0"/>
+        <geometry>
+          <box size="0.45 0.054 0.0001"/>
+        </geometry>
+      </collision>
+      <xacro:inertial_box mass="0.01" x="0.75" y="0.054" z="0.01">
+        <origin xyz="0 0 0"/>
+      </xacro:inertial_box>
+    </link>
+  </xacro:macro>
+  <!-- OBJECT-LINE JOINT LINK GENERATION -->
+  <xacro:macro name="line_to_obj" params="obj line *origin">
+    <xacro:make_line name="${line}"/>
+    <joint name="${obj}_${line}_joint" type="fixed">
+      <xacro:insert_block name="origin"/>
+      <parent link="${obj}"/>
+      <child link="${line}"/>
+    </joint>
+    <gazebo reference="${line}">
+      <material>Gazebo/Black</material>
+    </gazebo>
+  </xacro:macro>
 </robot>

File: world_desc/lks_arena.main.xacro (robot description, xacro)
@@ -38,4 +38,24 @@
   <xacro:wall_link name="wall_250_1" length="0.75" mass="0.75"/>
   <xacro:wall_link name="wall_750_0" length="2.25" mass="2.25"/>
+  <xacro:cont_box name="cont_box1"/>
+  <xacro:cont_box name="cont_box2"/>
+  <xacro:cont_box name="cont_box3"/>
+  <xacro:cont_box name="cont_box4"/>
+  <xacro:cont_box name="cont_box5"/>
+  <xacro:cont_box name="cont_box6"/>
+  <xacro:cont_box name="cont_box7"/>
+  <xacro:cont_box name="cont_box8"/>
+  <xacro:cont_box name="cont_box9"/>
+  <xacro:cont_box name="cont_box10"/>
+  <xacro:cont_box name="cont_box11"/>
+  <xacro:cont_box name="cont_box12"/>
+  <xacro:cont_box name="cont_box13"/>
+  <xacro:cont_box name="cont_box14"/>
+  <xacro:cont_box name="cont_box15"/>
+  <xacro:cont_box name="cont_box16"/>
+  <xacro:cont_box name="cont_box17"/>
+  <xacro:cont_box name="cont_box18"/>
+  <xacro:cont_box name="cont_box19"/>
+  <xacro:cont_box name="cont_box20"/>
   <xacro:wall_joint wall="wall_2000_0">
     <origin xyz="${plank_thick / 2 + 6} 0 ${wall_height / 2 + 0.027}" rpy="0 0 ${pi / 2}"/>
@@ -65,3 +85,111 @@
     <origin xyz="${-6 + 5.121} ${0.75 + 1.125} ${wall_height / 2 + 0.027}" rpy="0 0 ${pi / 2}"/>
   </xacro:wall_joint>
+  <xacro:cont_box_4
+    name0="cont_box1"
+    name1="cont_box2"
+    name2="cont_box3"
+    name3="cont_box4"
+    x="1.875"
+    y="0.75"
+  />
+  <xacro:cont_box_4
+    name0="cont_box5"
+    name1="cont_box6"
+    name2="cont_box7"
+    name3="cont_box8"
+    x="${1.875 + 2.379 + 0.6 + 0.15}"
+    y="1.575"
+  />
+  <xacro:cont_box_2
+    name0="cont_box9"
+    name1="cont_box10"
+    x="${1.8 + 0.054 + 2.271}"
+    y="${5.85 - 0.3}"
+  />
+  <xacro:cont_box_2
+    name0="cont_box11"
+    name1="cont_box12"
+    x="${1.8 + 0.054 + 2.271 + 0.6 + 0.15 + 1.125}"
+    y="${5.85 - 0.3}"
+  />
+  <xacro:cont_box_4
+    name0="cont_box13"
+    name1="cont_box14"
+    name2="cont_box15"
+    name3="cont_box16"
+    x="${1.8 + 0.054 + 2.271 + 0.6 * 2 + 0.15 * 2 + 1.125 + 0.75 + 0.054 + 1.821}"
+    y="${6 - 0.75 - 0.6 - 0.15}"
+  />
+    <xacro:cont_box_2
+    name0="cont_box17"
+    name1="cont_box18"
+    x="${1.8 + 0.054 + 2.271 + 0.6 * 2 + 0.15 * 2 + 1.125 + 0.75 + 0.054 + 1.821}"
+    y="${6 - 0.75 - 0.9 - 0.15 * 2}"
+  />
+  <xacro:wall_joint wall="cont_box19">
+    <origin xyz="${6 - (1.8 + 0.054 + 0.15) - 0.15} ${3 - (6 - 0.75 - 0.6 - 0.15) - 0.3 - 0.3} ${0.15 + 0.027}"/>
+  </xacro:wall_joint>
+  <xacro:wall_joint wall="cont_box20">
+    <origin xyz="${6 - (1.8 + 0.054 + 0.15) - 0.15} ${3 - (6 - 0.75 - 0.6 - 0.15) - 0.15} ${0.15 + 0.027}"/>
+  </xacro:wall_joint>
+  <xacro:line_to_obj obj="cont_box1" line="box1_line">
+    <origin xyz="${0.225 + 0.15} 0 -0.15" rpy="0 0 0"/>
+  </xacro:line_to_obj>
+  <xacro:line_to_obj obj="cont_box2" line="box2_line">
+    <origin xyz="${0.225 + 0.15} 0 -0.15" rpy="0 0 0"/>
+  </xacro:line_to_obj>
+  <xacro:line_to_obj obj="cont_box3" line="box3_line">
+    <origin xyz="-${0.225 + 0.15} 0 -0.15" rpy="0 0 0"/>
+  </xacro:line_to_obj>
+  <xacro:line_to_obj obj="cont_box4" line="box4_line">
+    <origin xyz="-${0.225 + 0.15} 0 -0.15" rpy="0 0 0"/>
+  </xacro:line_to_obj>
+  <xacro:line_to_obj obj="cont_box5" line="box5_line">
+    <origin xyz="0 -${0.225 + 0.15} -0.15" rpy="0 0 ${pi / 2}"/>
+  </xacro:line_to_obj>
+  <xacro:line_to_obj obj="cont_box6" line="box6_line">
+    <origin xyz="0 ${0.225 + 0.15} -0.15" rpy="0 0 ${pi / 2}"/>
+  </xacro:line_to_obj>
+  <xacro:line_to_obj obj="cont_box7" line="box7_line">
+    <origin xyz="0 ${0.225 + 0.15} -0.15" rpy="0 0 ${pi / 2}"/>
+  </xacro:line_to_obj>
+  <xacro:line_to_obj obj="cont_box8" line="box8_line">
+    <origin xyz="0 -${0.225 + 0.15} -0.15" rpy="0 0 ${pi / 2}"/>
+  </xacro:line_to_obj>
+  <xacro:line_to_obj obj="cont_box9" line="box9_line">
+    <origin xyz="0 ${0.225 + 0.15} -0.15" rpy="0 0 ${pi / 2}"/>
+  </xacro:line_to_obj>
+  <xacro:line_to_obj obj="cont_box10" line="box10_line">
+    <origin xyz="0 ${0.225 + 0.15} -0.15" rpy="0 0 ${pi / 2}"/>
+  </xacro:line_to_obj>
+  <xacro:line_to_obj obj="cont_box11" line="box11_line">
+    <origin xyz="0 ${0.225 + 0.15} -0.15" rpy="0 0 ${pi / 2}"/>
+  </xacro:line_to_obj>
+  <xacro:line_to_obj obj="cont_box12" line="box12_line">
+    <origin xyz="0 ${0.225 + 0.15} -0.15" rpy="0 0 ${pi / 2}"/>
+  </xacro:line_to_obj>
+  <xacro:line_to_obj obj="cont_box13" line="box13_line">
+    <origin xyz="${0.225 + 0.15} 0 -0.15" rpy="0 0 0"/>
+  </xacro:line_to_obj>
+  <xacro:line_to_obj obj="cont_box14" line="box14_line">
+    <origin xyz="${0.225 + 0.15} 0 -0.15" rpy="0 0 0"/>
+  </xacro:line_to_obj>
+  <xacro:line_to_obj obj="cont_box15" line="box15_line">
+    <origin xyz="-${0.225 + 0.15} 0 -0.15" rpy="0 0 0"/>
+  </xacro:line_to_obj>
+  <xacro:line_to_obj obj="cont_box16" line="box16_line">
+    <origin xyz="-${0.225 + 0.15} 0 -0.15" rpy="0 0 0"/>
+  </xacro:line_to_obj>
+  <xacro:line_to_obj obj="cont_box17" line="box17_line">
+    <origin xyz="${0.225 + 0.15} 0 -0.15" rpy="0 0 0"/>
+  </xacro:line_to_obj>
+  <xacro:line_to_obj obj="cont_box18" line="box18_line">
+    <origin xyz="-${0.225 + 0.15} 0 -0.15" rpy="0 0 0"/>
+  </xacro:line_to_obj>
+  <xacro:line_to_obj obj="cont_box19" line="box19_line">
+    <origin xyz="-${0.225 + 0.15} 0 -0.15" rpy="0 0 0"/>
+  </xacro:line_to_obj>
+  <xacro:line_to_obj obj="cont_box20" line="box20_line">
+    <origin xyz="-${0.225 + 0.15} 0 -0.15" rpy="0 0 0"/>
+  </xacro:line_to_obj>
 </robot>

Commit message: Added racks and home line, reorder launch file

File: world_desc/lks_arena.include.xacro (robot description, xacro)
@@ -12,4 +12,38 @@
               izz="${(1/12) * mass * (x*x+y*y)}" />
     </inertial>
+  </xacro:macro>
+  <!-- PLANK GENERATION -->
+  <xacro:macro name="make_plank" params="name length width mass">
+    <link name="${name}">
+      <visual>
+        <origin xyz="0 0 0"/>
+        <geometry>
+          <box size="${length} ${plank_thick} ${width}"/>
+        </geometry>
+        <material name="white">
+          <color rgba="1 1 1 1"/>
+        </material>
+      </visual>
+      <collision>
+        <origin xyz="0 0 0"/>
+        <geometry>
+          <box size="${length} ${plank_thick} ${width}"/>
+        </geometry>
+      </collision>
+      <xacro:inertial_box mass="${mass}" x="${length}" y="${plank_thick}" z="${width}">
+        <origin xyz="0 0 0"/>
+      </xacro:inertial_box>
+    </link>
+    <gazebo reference="${name}">
+      <material>Gazebo/White</material>
+    </gazebo>
+  </xacro:macro>
+  <!-- OBJECT-OBJECT JOINT GENERATION -->
+  <xacro:macro name="obj_to_obj" params="name0 name1 *origin">
+    <joint name="${name0}_${name1}_joint" type="fixed">
+      <xacro:insert_block name="origin"/>
+      <parent link="${name0}"/>
+      <child link="${name1}"/>
+    </joint>
   </xacro:macro>
   <!-- WALL GENERATION -->

File: world_desc/lks_arena.main.xacro (robot description, xacro)
@@ -29,8 +29,9 @@
       <material>Gazebo/White</material>
     </gazebo>
+  <!-- WALL LINKS -->
   <xacro:wall_link name="wall_2000_0" length="6" mass="6"/>
   <xacro:wall_link name="wall_2000_1" length="6" mass="6"/>
   <xacro:wall_link name="wall_4000_0" length="12" mass="12"/>
-  <xacro:wall_link name="wall_4000_1" length="12" mass="12"/>
+  <xacro:make_plank name="wall_4000_1" length="12" width="1.2" mass="12"/>
   <xacro:wall_link name="wall_500_0" length="1.5" mass="1.5"/>
   <xacro:wall_link name="wall_500_1" length="1.5" mass="1.5"/>
@@ -38,4 +39,137 @@
   <xacro:wall_link name="wall_250_1" length="0.75" mass="0.75"/>
   <xacro:wall_link name="wall_750_0" length="2.25" mass="2.25"/>
+  <link name="home_line_0">
+    <visual>
+      <origin xyz="0 0 0"/>
+      <geometry>
+        <box size="1.8 0.054 0.0001"/>
+      </geometry>
+      <material name="black">
+        <color rgba="0.01 0.01 0.01 1"/>
+      </material>
+    </visual>
+    <collision>
+      <origin xyz="0 0 0"/>
+      <geometry>
+        <box size="1.8 0.054 0.0001"/>
+      </geometry>
+    </collision>
+    <xacro:inertial_box mass="0.01" x="0.75" y="0.054" z="0.01">
+      <origin xyz="0 0 0"/>
+    </xacro:inertial_box>
+  </link>
+  <link name="home_line_1">
+    <visual>
+      <origin xyz="0 0 0"/>
+      <geometry>
+        <box size="1.8 0.054 0.0001"/>
+      </geometry>
+      <material name="black">
+        <color rgba="0.01 0.01 0.01 1"/>
+      </material>
+    </visual>
+    <collision>
+      <origin xyz="0 0 0"/>
+      <geometry>
+        <box size="1.8 0.054 0.0001"/>
+      </geometry>
+    </collision>
+    <xacro:inertial_box mass="0.01" x="0.75" y="0.054" z="0.01">
+      <origin xyz="0 0 0"/>
+    </xacro:inertial_box>
+  </link>
+  <link name="home_line_2">
+    <visual>
+      <origin xyz="0 0 0"/>
+      <geometry>
+        <box size="1.8 0.054 0.0001"/>
+      </geometry>
+      <material name="black">
+        <color rgba="0.01 0.01 0.01 1"/>
+      </material>
+    </visual>
+    <collision>
+      <origin xyz="0 0 0"/>
+      <geometry>
+        <box size="1.8 0.054 0.0001"/>
+      </geometry>
+    </collision>
+    <xacro:inertial_box mass="0.01" x="0.75" y="0.054" z="0.01">
+      <origin xyz="0 0 0"/>
+    </xacro:inertial_box>
+  </link>
+  <link name="home_line_3">
+    <visual>
+      <origin xyz="0 0 0"/>
+      <geometry>
+        <box size="1.8 0.054 0.0001"/>
+      </geometry>
+      <material name="black">
+        <color rgba="0.01 0.01 0.01 1"/>
+      </material>
+    </visual>
+    <collision>
+      <origin xyz="0 0 0"/>
+      <geometry>
+        <box size="1.8 0.054 0.0001"/>
+      </geometry>
+    </collision>
+    <xacro:inertial_box mass="0.01" x="0.75" y="0.054" z="0.01">
+      <origin xyz="0 0 0"/>
+    </xacro:inertial_box>
+  </link>
+  <!-- WALL JOINTS -->
+  <xacro:wall_joint wall="wall_2000_0">
+    <origin xyz="${plank_thick / 2 + 6} 0 ${wall_height / 2 + 0.027}" rpy="0 0 ${pi / 2}"/>
+  </xacro:wall_joint>
+  <xacro:wall_joint wall="wall_2000_1">
+    <origin xyz="${-plank_thick / 2 - 6} 0 ${wall_height / 2 + 0.027}" rpy="0 0 ${pi / 2}"/>
+  </xacro:wall_joint>
+  <xacro:wall_joint wall="wall_4000_0">
+    <origin xyz="0 ${-plank_thick / 2 - 3} ${wall_height / 2 + 0.027}"/>
+  </xacro:wall_joint>
+  <xacro:wall_joint wall="wall_4000_1">
+    <origin xyz="0 ${plank_thick / 2 + 3} ${1.2 / 2 + 0.027}"/>
+  </xacro:wall_joint>
+  <xacro:wall_joint wall="wall_500_0">
+    <origin xyz="${6 - 1.8} ${-3 + 0.75} ${wall_height / 2 + 0.027}" rpy="0 0 ${pi / 2}"/>
+  </xacro:wall_joint>
+  <xacro:wall_joint wall="wall_500_1">
+    <origin xyz="${-6 + 0.75} 0.75 ${wall_height / 2 + 0.027}"/>
+  </xacro:wall_joint>
+  <xacro:wall_joint wall="wall_250_0">
+    <origin xyz="${-6 + 4.446} ${-3 + 0.375} ${wall_height / 2 + 0.027}" rpy="0 0 ${pi / 2}"/>
+  </xacro:wall_joint>
+  <xacro:wall_joint wall="wall_250_1">
+    <origin xyz="${-6 + 5.121} 0.75 ${wall_height / 2 + 0.027}"/>
+  </xacro:wall_joint>
+  <xacro:wall_joint wall="wall_750_0">
+    <origin xyz="${-6 + 5.121} ${0.75 + 1.125} ${wall_height / 2 + 0.027}" rpy="0 0 ${pi / 2}"/>
+  </xacro:wall_joint>
+  <xacro:obj_to_obj name0="wall_500_0" name1="home_line_0">
+    <origin xyz="${0.1 + 0.054} -${0.054} -0.3"/>
+  </xacro:obj_to_obj>
+  <xacro:obj_to_obj name0="wall_500_0" name1="home_line_1">
+    <origin xyz="${0.1 + 0.054} -${1.8 - 0.027} -0.3"/>
+  </xacro:obj_to_obj>
+  <xacro:obj_to_obj name0="wall_500_0" name1="home_line_2">
+    <origin xyz="${0.1 + 0.054 - 0.9 + 0.027} -${0.9 + 0.027} -0.3" rpy="0 0 ${pi / 2}"/>
+  </xacro:obj_to_obj>
+  <xacro:obj_to_obj name0="wall_500_0" name1="home_line_3">
+    <origin xyz="${0.1 + 0.054 - 0.9 + 0.027 + 1.8} -${0.9 + 0.027} -0.3" rpy="0 0 ${pi / 2}"/>
+  </xacro:obj_to_obj>
+  <gazebo reference="home_line_0">
+    <material>Gazebo/Black</material>
+  </gazebo>
+  <gazebo reference="home_line_1">
+    <material>Gazebo/Black</material>
+  </gazebo>
+  <gazebo reference="home_line_2">
+    <material>Gazebo/Black</material>
+  </gazebo>
+  <gazebo reference="home_line_3">
+    <material>Gazebo/Black</material>
+  </gazebo>
+  <!-- CONTAINER BOXES LINKS -->
   <xacro:cont_box name="cont_box1"/>
   <xacro:cont_box name="cont_box2"/>
@@ -58,31 +192,5 @@
   <xacro:cont_box name="cont_box19"/>
   <xacro:cont_box name="cont_box20"/>
-  <xacro:wall_joint wall="wall_2000_0">
-    <origin xyz="${plank_thick / 2 + 6} 0 ${wall_height / 2 + 0.027}" rpy="0 0 ${pi / 2}"/>
-  </xacro:wall_joint>
-  <xacro:wall_joint wall="wall_2000_1">
-    <origin xyz="${-plank_thick / 2 - 6} 0 ${wall_height / 2 + 0.027}" rpy="0 0 ${pi / 2}"/>
-  </xacro:wall_joint>
-  <xacro:wall_joint wall="wall_4000_0">
-    <origin xyz="0 ${-plank_thick / 2 - 3} ${wall_height / 2 + 0.027}"/>
-  </xacro:wall_joint>
-  <xacro:wall_joint wall="wall_4000_1">
-    <origin xyz="0 ${plank_thick / 2 + 3} ${wall_height / 2 + 0.027}"/>
-  </xacro:wall_joint>
-  <xacro:wall_joint wall="wall_500_0">
-    <origin xyz="${6 - 1.8} ${-3 + 0.75} ${wall_height / 2 + 0.027}" rpy="0 0 ${pi / 2}"/>
-  </xacro:wall_joint>
-  <xacro:wall_joint wall="wall_500_1">
-    <origin xyz="${-6 + 0.75} 0.75 ${wall_height / 2 + 0.027}"/>
-  </xacro:wall_joint>
-  <xacro:wall_joint wall="wall_250_0">
-    <origin xyz="${-6 + 4.446} ${-3 + 0.375} ${wall_height / 2 + 0.027}" rpy="0 0 ${pi / 2}"/>
-  </xacro:wall_joint>
-  <xacro:wall_joint wall="wall_250_1">
-    <origin xyz="${-6 + 5.121} 0.75 ${wall_height / 2 + 0.027}"/>
-  </xacro:wall_joint>
-  <xacro:wall_joint wall="wall_750_0">
-    <origin xyz="${-6 + 5.121} ${0.75 + 1.125} ${wall_height / 2 + 0.027}" rpy="0 0 ${pi / 2}"/>
-  </xacro:wall_joint>
+  <!-- CONTAINER BOXES CLUSTERS -->
   <xacro:cont_box_4
     name0="cont_box1"
@@ -133,4 +241,5 @@
     <origin xyz="${6 - (1.8 + 0.054 + 0.15) - 0.15} ${3 - (6 - 0.75 - 0.6 - 0.15) - 0.15} ${0.15 + 0.027}"/>
   </xacro:wall_joint>
+  <!-- CONTAINER BOXES JOINTS -->
   <xacro:line_to_obj obj="cont_box1" line="box1_line">
     <origin xyz="${0.225 + 0.15} 0 -0.15" rpy="0 0 0"/>
@@ -193,3 +302,95 @@
     <origin xyz="-${0.225 + 0.15} 0 -0.15" rpy="0 0 0"/>
   </xacro:line_to_obj>
+  <!-- BOX RACK LINKS -->
+  <xacro:make_plank name="box_rack_plank_0" width="1.443" length="0.3" mass="0.3"/>
+  <xacro:make_plank name="box_rack_plank_1" width="1.443" length="0.3" mass="0.3"/>
+  <xacro:make_plank name="box_rack_plank_2" width="1.293" length="0.3" mass="0.3"/>
+  <xacro:make_plank name="box_rack_plank_3" width="1.185" length="0.3" mass="0.3"/>
+  <xacro:make_plank name="box_rack_plank_4" width="1.185" length="0.3" mass="0.3"/>
+  <xacro:make_plank name="box_rack_plank_5" width="1.185" length="0.3" mass="0.3"/>
+  <xacro:make_line name="box_rack_line_0"/>
+  <xacro:make_line name="box_rack_line_1"/>
+  <xacro:make_line name="box_rack_line_2"/>
+  <!-- BOX RACK JOINTS -->
+  <xacro:obj_to_obj name0="box_rack_plank_0" name1="box_rack_plank_1">
+    <origin xyz="0 ${1.185 + 0.054} 0"/>
+  </xacro:obj_to_obj>
+  <xacro:obj_to_obj name0="box_rack_plank_1" name1="box_rack_plank_2">
+    <origin xyz="0 -0.6195 ${1.443 / 2}" rpy="${pi / 2} 0 0"/>
+  </xacro:obj_to_obj>
+  <xacro:obj_to_obj name0="box_rack_plank_2" name1="box_rack_plank_3">
+    <origin xyz="0 -${0.345 + 0.054} 0" rpy="0 0 0"/>
+  </xacro:obj_to_obj>
+  <xacro:obj_to_obj name0="box_rack_plank_3" name1="box_rack_plank_4">
+    <origin xyz="0 -${0.345 + 0.054} 0" rpy="0 0 0"/>
+  </xacro:obj_to_obj>
+  <xacro:obj_to_obj name0="box_rack_plank_4" name1="box_rack_plank_5">
+    <origin xyz="0 -${0.345 + 0.054} 0" rpy="0 0 0"/>
+  </xacro:obj_to_obj>
+  <xacro:obj_to_obj name0="box_rack_plank_5" name1="box_rack_line_0">
+    <origin xyz="${-0.225 - 0.3} -${0.3 - 0.054} 0" rpy="${pi / 2} 0 0"/>
+  </xacro:obj_to_obj>
+  <xacro:obj_to_obj name0="box_rack_plank_5" name1="box_rack_line_1">
+    <origin xyz="${-0.225 - 0.3} -${0.3 - 0.054} 0.345" rpy="${pi / 2} 0 0"/>
+  </xacro:obj_to_obj>
+  <xacro:obj_to_obj name0="box_rack_plank_5" name1="box_rack_line_2">
+    <origin xyz="${-0.225 - 0.3} -${0.3 - 0.054} -0.345" rpy="${pi / 2} 0 0"/>
+  </xacro:obj_to_obj>
+  <xacro:wall_joint wall="box_rack_plank_0">
+    <origin xyz="${-6 - 0.027 + 2.043} ${3 - 0.15} 0.7485" rpy="0 0 ${pi / 2}"/>
+  </xacro:wall_joint>
+  <!-- DRINK RACK LINKS -->
+  <link name="drink_rack">
+      <visual>
+        <origin xyz="0 0 0"/>
+        <geometry>
+          <mesh
+            filename="file://$(find mecabot_gz)/../../../../world_desc/mesh/drink_rack.stl"
+            scale="1.5 1.5 1.5"
+          />
+        </geometry>
+        <material name="white">
+          <color rgba="1 1 1 1"/>
+        </material>
+      </visual>
+      <collision>
+        <origin xyz="0 0 0"/>
+        <geometry>
+          <mesh
+            filename="file://$(find mecabot_gz)/../../../../world_desc/mesh/drink_rack.stl"
+            scale="1.5 1.5 1.5"
+          />
+        </geometry>
+      </collision>
+      <xacro:inertial_box mass="1.5" x="1.6" y="0.3" z="1">
+        <origin xyz="0 0 0"/>
+      </xacro:inertial_box>
+  </link>
+  <gazebo reference="drink_rack">
+    <material>Gazebo/White</material>
+  </gazebo>
+  <xacro:make_line name="drink_rack_line_0"/>
+  <xacro:make_line name="drink_rack_line_1"/>
+  <xacro:make_line name="drink_rack_line_2"/>
+  <xacro:make_line name="drink_rack_line_3"/>
+  <xacro:make_line name="drink_rack_line_4"/>
+  <!-- DRINK RACK JOINTS -->
+  <xacro:wall_joint wall="drink_rack">
+    <origin xyz="${-6 + 0.789 + 0.002 + 2.793} ${3 - 0.108 - 0.027} 0.027" rpy="0 0 0"/>
+  </xacro:wall_joint>
+  <xacro:obj_to_obj name0="drink_rack" name1="drink_rack_line_0">
+    <origin xyz="0 ${-0.225 * 2 - 0.15} 0" rpy="0 0 ${pi / 2}"/>
+  </xacro:obj_to_obj>
+  <xacro:obj_to_obj name0="drink_rack" name1="drink_rack_line_1">
+    <origin xyz="0.2502 ${-0.225 * 2 - 0.15} 0" rpy="0 0 ${pi / 2}"/>
+  </xacro:obj_to_obj>
+  <xacro:obj_to_obj name0="drink_rack" name1="drink_rack_line_2">
+    <origin xyz="${0.2502 * 2} ${-0.225 * 2 - 0.15} 0" rpy="0 0 ${pi / 2}"/>
+  </xacro:obj_to_obj>
+  <xacro:obj_to_obj name0="drink_rack" name1="drink_rack_line_3">
+    <origin xyz="-0.2502 ${-0.225 * 2 - 0.15} 0" rpy="0 0 ${pi / 2}"/>
+  </xacro:obj_to_obj>
+  <xacro:obj_to_obj name0="drink_rack" name1="drink_rack_line_4">
+    <origin xyz="-${0.2502 * 2} ${-0.225 * 2 - 0.15} 0" rpy="0 0 ${pi / 2}"/>
+  </xacro:obj_to_obj>
 </robot>

Commit message: Added props spawner xacro file

File: world_desc/lks_arena.include.xacro (robot description, xacro)
@@ -11,4 +11,14 @@
               iyy="${(1/12) * mass * (x*x+z*z)}" iyz="0.0"
               izz="${(1/12) * mass * (x*x+y*y)}" />
+    </inertial>
+  </xacro:macro>
+  <!-- CYLINDER INERTIA MACRO -->
+  <xacro:macro name="inertial_cylinder" params="mass length radius *origin">
+    <inertial>
+      <xacro:insert_block name="origin"/>
+      <mass value="${mass}" />
+      <inertia ixx="${(1/12) * mass * (3*radius*radius + length*length)}" ixy="0.0" ixz="0.0"
+              iyy="${(1/12) * mass * (3*radius*radius + length*length)}" iyz="0.0"
+              izz="${(1/2) * mass * (radius*radius)}" />
     </inertial>
   </xacro:macro>
