Commit message: Fixed card bug, adjusted sizes

File: world_desc/lks_arena.spawnprops.xacro (robot description, xacro)
@@ -75,5 +75,5 @@
         <geometry>
           <!-- Assuming container box length -->
-          <cylinder radius="0.28" length="0.0001"/>
+          <cylinder radius="0.14" length="0.001"/>
         </geometry>
         <material name="$(arg color)"/>
@@ -83,8 +83,8 @@
         <geometry>
           <!-- Assuming container box length -->
-          <cylinder radius="0.28" length="0.0001"/>
+          <cylinder radius="0.14" length="0.001"/>
         </geometry>
       </collision>
-      <xacro:inertial_cylinder mass="0.001" length="0.0001" radius="0.28">
+      <xacro:inertial_cylinder mass="0.001" length="0.001" radius="0.28">
         <origin xyz="0 0 0"/>
       </xacro:inertial_cylinder>
@@ -98,5 +98,5 @@
         <geometry>
           <!-- Assuming container box length -->
-          <box size="0.28 0.28 0.000"/>
+          <box size="0.28 0.28 0.001"/>
         </geometry>
         <material name="$(arg color)"/>
@@ -106,8 +106,8 @@
         <geometry>
           <!-- Assuming container box length -->
-          <box size="0.28 0.28 0.0001"/>
+          <box size="0.28 0.28 0.001"/>
         </geometry>
       </collision>
-      <xacro:inertial_box mass="0.001" x="0.28" y="0.28" z="0.0001">
+      <xacro:inertial_box mass="0.001" x="0.28" y="0.28" z="0.001">
         <origin xyz="0 0 0"/>
       </xacro:inertial_box>
