Commit message: Readjust physics, longer launch delay

File: robot_desc/mecabot_gz.include.xacro (robot description, xacro)
@@ -40,12 +40,12 @@
       <inertial>
         <!-- Values from Gazebo Harmonic mecanum_drive.sdf -->
-        <mass value="1"/>
+        <mass value="0.5"/>
         <inertia
-          ixx="0.072916"
+          ixx="0.036458"
           ixy="0"
           ixz="0"
-          iyy="0.072916"
+          iyy="0.036458"
           iyz="0"
-          izz="0.0625"
+          izz="0.03125"
         />
       </inertial>
@@ -61,5 +61,5 @@
             <ode>
               <mu>1.5</mu>
-              <mu2>0</mu2>
+              <mu2>0.5</mu2>
               <xacro:if value="${direction == 'left'}">
                 <fdir1 gz:expressed_in="base_link">1 -1 0</fdir1>

File: robot_desc/mecabot_gz.main.xacro (robot description, xacro)
@@ -20,5 +20,5 @@
       </geometry>
     </collision>
-    <xacro:inertial_box mass="5" x="${base_link_x}" y="${base_link_y}" z="${base_link_z}">
+    <xacro:inertial_box mass="3" x="${base_link_x}" y="${base_link_y}" z="${base_link_z}">
       <origin />
     </xacro:inertial_box>

Commit message: Implemented ros2_control joint states, built previously unbuilt directories

File: robot_desc/mecabot_gz.include.xacro (robot description, xacro)
@@ -26,5 +26,5 @@
         <geometry>
           <mesh
-            filename="file://$(find mecabot_gz)/../../../../robot_desc/mesh/mecanum_${direction}.STL"
+            filename="file://$(find mecabot_gz)/robot_desc/mesh/mecanum_${direction}.STL"
             scale="${mecanum_radius * 2 / 100} ${mecanum_radius * 2 / 100} ${mecanum_radius * 2 / 100}"
           /> <!-- Scale mesh to radius -->
@@ -82,5 +82,5 @@
         <geometry>
           <mesh
-            filename="file://$(find mecabot_gz)/../../../../robot_desc/mesh/omni_wheel.stl"
+            filename="file://$(find mecabot_gz)/robot_desc/mesh/omni_wheel.stl"
             scale="${omni_radius / 5} ${omni_radius / 5} ${omni_radius / 5}"
           /> <!-- Scale mesh to radius -->

File: robot_desc/mecabot_gz.main.xacro (robot description, xacro)
@@ -129,8 +129,38 @@
     </plugin>
     <plugin
-      filename="gz-sim-joint-state-publisher-system"
-      name="gz::sim::systems::JointStatePublisher">
-      <topic>/joint_states</topic>
+      name="gz_ros2_control::GazeboSimROS2ControlPlugin"
+      filename="libgz_ros2_control-system">
+      <parameters>$(find mecabot_gz)/config/test_controller.yaml</parameters>
     </plugin>
   </gazebo>
+  <!-- ROS2 Control -->
+  <ros2_control name="GazeboSimSystem" type="system">
+    <hardware>
+      <plugin>gz_ros2_control/GazeboSimSystem</plugin>
+    </hardware>
+    <joint name="y_front_omni_joint">
+      <state_interface name="position"/>
+    </joint>
+    <joint name="y_rear_omni_joint">
+      <state_interface name="position"/>
+    </joint>
+    <joint name="x_right_omni_joint">
+      <state_interface name="position"/>
+    </joint>
+    <joint name="x_left_omni_joint">
+      <state_interface name="position"/>
+    </joint>
+    <joint name="front_left_mecanum_joint">
+      <state_interface name="position"/>
+    </joint>
+    <joint name="front_right_mecanum_joint">
+      <state_interface name="position"/>
+    </joint>
+    <joint name="rear_left_mecanum_joint">
+      <state_interface name="position"/>
+    </joint>
+    <joint name="rear_right_mecanum_joint">
+      <state_interface name="position"/>
+    </joint>
+  </ros2_control>
 </robot>

File: world_desc/lks_arena.main.xacro (robot description, xacro)
@@ -346,5 +346,5 @@
         <geometry>
           <mesh
-            filename="file://$(find mecabot_gz)/../../../../world_desc/mesh/drink_rack.stl"
+            filename="file://$(find mecabot_gz)/world_desc/mesh/drink_rack.stl"
             scale="1.5 1.5 1.5"
           />
@@ -358,5 +358,5 @@
         <geometry>
           <mesh
-            filename="file://$(find mecabot_gz)/../../../../world_desc/mesh/drink_rack.stl"
+            filename="file://$(find mecabot_gz)/world_desc/mesh/drink_rack.stl"
             scale="1.5 1.5 1.5"
           />
