Commit message: Removed rear omni wheel, extended omni gap for better readings

File: robot_desc/mecabot_gz.main.xacro (robot description, xacro)
@@ -41,7 +41,4 @@
     <material name="grey"/>
   </xacro:gen_omni_wheel>
-  <xacro:gen_omni_wheel name="y_rear_omni">
-    <material name="grey"/>
-  </xacro:gen_omni_wheel>
   <xacro:gen_omni_wheel name="x_right_omni">
     <material name="grey"/>
@@ -51,5 +48,5 @@
   </xacro:gen_omni_wheel>
   <!-- OMNI WHEEL JOINTS -->
-  <xacro:property name="omni_gap" value="0.15"/>
+  <xacro:property name="omni_gap" value="0.4"/>
   <xacro:property name="omni_joint_friction" value="0.1"/>
   <xacro:property name="omni_joint_damping" value="0"/>
@@ -72,11 +69,4 @@
     <parent link="base_link"/>
     <child link="x_left_omni_link"/>
-    <axis xyz="0 1 0"/>
-    <dynamics damping="${omni_joint_damping}" friction="${omni_joint_friction}"/>
-  </joint>
-  <joint name="y_rear_omni_joint" type="continuous">
-    <origin xyz="-${omni_gap} 0 ${omni_radius - mecanum_radius}" rpy="0 0 ${pi / 2}"/>
-    <parent link="base_link"/>
-    <child link="y_rear_omni_link"/>
     <axis xyz="0 1 0"/>
     <dynamics damping="${omni_joint_damping}" friction="${omni_joint_friction}"/>
@@ -142,7 +132,4 @@
       <state_interface name="position"/>
     </joint>
-    <joint name="y_rear_omni_joint">
-      <state_interface name="position"/>
-    </joint>
     <joint name="x_right_omni_joint">
       <state_interface name="position"/>
